Commit message: Set the IMU yaw to +90, as measured on the car
Verified by rotating the car counter-clockwise and watching
angular_velocity.z go positive. It was -90, which would have inverted every
rotation cartographer and the EKF see.

Leaves an open question in the joint comment rather than guessing at it: the
board's Z axis reportedly faces the floor, and a Z flip is a roll of pi, not a
rotation about the vertical, so yaw alone may not describe the mounting. That
matters separately from the yaw sign because cartographer uses the IMU to find
which way is down. The check is one command with the car level and still, and
it is in the comment and in README's TODO.

Co-Authored-By: Claude Opus 5 <noreply@anthropic.com>

File: src/albomb_description/urdf/albomb_sensors.xacro (robot description, xacro)
@@ -10,8 +10,20 @@
     </visual>
   </link>
+  <!-- VESC 6 MkVI onboard IMU.
+       Yaw is +90 deg, verified on the car: rotating it counter-clockwise gives
+       a positive angular_velocity.z on /vesc/sensors/imu/raw. It was -90 here
+       until then, which would have inverted every rotation the filters see.
+       OPEN: the board's Z axis reportedly points at the floor. If that is so,
+       yaw alone does not describe the mounting - a Z flip is a roll or pitch of
+       pi, not a rotation about the vertical - and this joint is still wrong for
+       gravity. It matters because cartographer uses the IMU to find "down", and
+       an inverted Z makes it find "up". Check with the car level and still:
+           ros2 topic echo /vesc/sensors/imu/raw --field linear_acceleration
+       z should read about +9.8. If it reads about -9.8, add rpy roll=pi here
+       and re-verify the yaw sign afterwards, since the flip changes it. -->
   <joint name="imu_joint" type="fixed">
     <parent link="${car_name}/base_link"/>
     <child link="${car_name}/imu"/>
-    <origin xyz="0.07 0.0 ${wheel_radius+0.04}" rpy="0 0 -1.5708"/>
+    <origin xyz="0.07 0.0 ${wheel_radius+0.04}" rpy="0 0 1.5708"/>
   </joint>
   <link name="${car_name}/laser">

Commit message: Flip the IMU joint to match the board: Z faces the floor
rpy 0 0 1.5708 -> 3.141592 0 1.5708, established on the car. With both
rotations the axes come out as forward = +imu.y, left = +imu.x, up = -imu.z,
so the yaw rate is -angular_velocity.z - exactly what UNIST hardcoded for
their own car, which is a second and independent sign this is right.

Corrects the comment this file carried until now, which read VESC Tool's Imu
Rotation Roll of 7.4 degrees as proof that Z was up. That value is mounting
tilt applied inside the firmware and says nothing about which way the board
faces in the data we receive.

No controller change needed: controller_manager now takes this rotation from
TF, so it follows the URDF.

Cartographer tracks in this frame, so until now its IMU and its laser scans
disagreed about which way yaw ran. Maps already saved were built that way.

Co-Authored-By: Claude Opus 5 <noreply@anthropic.com>

File: src/albomb_description/urdf/albomb_sensors.xacro (robot description, xacro)
@@ -10,18 +10,22 @@
     </visual>
   </link>
-  <!-- VESC 6 MkVI onboard IMU. Yaw +90 deg, verified on the car by rotating it
-       counter-clockwise and watching angular_velocity.z go positive.
-       Z is up, not down: VESC Tool's IMU calibration levelled the board with
-       roll 7.4 deg and pitch -4.7 deg, which is mounting tilt. A board facing
-       the floor would have needed roll near 180. Its Imu Rotation Yaw is 0, so
-       the +90 here is the only place the yaw is applied - do not also set it
-       in the firmware or it lands twice.
+  <!-- VESC 6 MkVI onboard IMU: yaw +90 deg and Z facing the floor, both
+       established on the car.
+       Roll pi is the Z flip, not a tilt. Together the two give
+           forward = +imu.y    left = +imu.x    up = -imu.z
+       so level and still, imu.z reads about -9.8, and the yaw rate is
+       -angular_velocity.z. That last one is what UNIST hardcoded for their own
+       car, which is a second, independent sign that this is the right way up.
+       VESC Tool's own Imu Rotation is roll 7.4 / pitch -4.7 / yaw 0 - mounting
+       tilt only. Do not put the 90 or the 180 in there as well; this joint is
+       where they belong, and the firmware would apply them twice.
        This joint is the single description of the mounting. controller_manager
-       reads it back through TF to rotate the IMU into the car's axes, so
-       getting it wrong here silently rotates the controller's yaw rate too. -->
+       reads it back through TF to rotate the IMU into the car's axes, and
+       cartographer tracks in this frame, so an error here rotates the
+       controller's yaw rate and tilts the map with no other symptom. -->
   <joint name="imu_joint" type="fixed">
     <parent link="${car_name}/base_link"/>
     <child link="${car_name}/imu"/>
-    <origin xyz="0.07 0.0 ${wheel_radius+0.04}" rpy="0 0 1.5708"/>
+    <origin xyz="0.07 0.0 ${wheel_radius+0.04}" rpy="3.141592 0 1.5708"/>
   </joint>
   <link name="${car_name}/laser">

Commit message: Revert the IMU roll: the data is Z up, whatever the chip is doing
Measured on the car, level and still, on /vesc/sensors/imu/raw:

    linear_acceleration:  x 0.139   y 0.082   z 9.910

An accelerometer at rest reads the reaction to gravity, so +9.9 on z is z
pointing up. That topic is published by the driver and never passes through
the URDF, so the reading is the same with or without roll=pi - which is what
makes it a measurement of the sensor frame rather than of what we assert
about it.

The chip really is mounted upside down; the firmware already corrects for it.
The URDF has to describe the data we receive, not the silicon, so roll=pi
applied the flip a second time. Back to rpy="0 0 1.5708".

This also restores agreement with the earlier check that rotating the car
counter-clockwise drives angular_velocity.z positive, which needs z up.

Still unverified, and untestable from a static reading: +90 against -90. It
sets the longitudinal axis only, not the yaw rate. Recorded in the file with
the test - push the car forward and imu.y should go negative.

Co-Authored-By: Claude Opus 5 <noreply@anthropic.com>

File: src/albomb_description/urdf/albomb_sensors.xacro (robot description, xacro)
@@ -10,14 +10,24 @@
     </visual>
   </link>
-  <!-- VESC 6 MkVI onboard IMU: yaw +90 deg and Z facing the floor, both
-       established on the car.
-       Roll pi is the Z flip, not a tilt. Together the two give
-           forward = +imu.y    left = +imu.x    up = -imu.z
-       so level and still, imu.z reads about -9.8, and the yaw rate is
-       -angular_velocity.z. That last one is what UNIST hardcoded for their own
-       car, which is a second, independent sign that this is the right way up.
-       VESC Tool's own Imu Rotation is roll 7.4 / pitch -4.7 / yaw 0 - mounting
-       tilt only. Do not put the 90 or the 180 in there as well; this joint is
-       where they belong, and the firmware would apply them twice.
+  <!-- VESC 6 MkVI onboard IMU. Yaw +90 deg; no roll.
+       The chip is mounted upside down on the board, but the FIRMWARE already
+       corrects for that, so the data reaching us is Z up. Measured, level and
+       still, on /vesc/sensors/imu/raw:
+           linear_acceleration:  x 0.139   y 0.082   z 9.910
+       An accelerometer at rest reads the reaction to gravity, so +9.9 on z is
+       z pointing up; a flipped frame would read -9.9. That topic comes
+       straight from the driver and never passes through this file, which is
+       what makes it a clean measurement of the sensor frame rather than of
+       what we claim about it. Adding roll=pi here describes the chip instead
+       of the data and applies the flip a second time.
+       So: up = +imu.z, and the yaw rate is +angular_velocity.z. That agrees
+       with the earlier check of rotating the car counter-clockwise and
+       watching angular_velocity.z go positive.
+       STILL UNVERIFIED is +90 vs -90, which this static reading cannot show
+       and which only sets the longitudinal axis, not the yaw rate. At +90,
+       forward = -imu.y, so accelerating forwards should drive imu.y negative.
+       If it goes positive, this is -1.5708.
+       VESC Tool's own Imu Rotation (roll 7.4 / pitch -4.7 / yaw 0) is mounting
+       tilt only. Leave the 90 out of it; this joint is where it belongs.
        This joint is the single description of the mounting. controller_manager
        reads it back through TF to rotate the IMU into the car's axes, and
@@ -27,5 +37,5 @@
     <parent link="${car_name}/base_link"/>
     <child link="${car_name}/imu"/>
-    <origin xyz="0.07 0.0 ${wheel_radius+0.04}" rpy="3.141592 0 1.5708"/>
+    <origin xyz="0.07 0.0 ${wheel_radius+0.04}" rpy="0 0 1.5708"/>
   </joint>
   <link name="${car_name}/laser">

Commit message: IMU yaw is -90: the board is turned clockwise from the car's forward axis
Physical inspection: the VESC sits 90 degrees CLOCKWISE relative to the car's
forward direction, so the imu frame is -90 about z from base_link. rpy rotates
child vectors into the parent, so the sign follows directly.

This was the original value. It became +1.5708 while Z was believed to face
the floor, and that was self-consistent at the time: Rz(+90)Rx(180) and
Rz(-90) produce the same forward axis. Once the accelerometer showed Z up, the
roll went away and this is what is left.

Nothing measured so far contradicts it. A yaw rotation leaves z alone, so the
gyro check that pinned Z up cannot distinguish +90 from -90; the outstanding
test is pushing the car forwards, where imu.y should now go positive.

Cartographer is unaffected either way - it tracks in the imu frame and
publishes base_link, so a constant imu/laser rotation is applied and removed,
and 2D uses only gyro z. Maps made before this are still good.
controller_manager does read the longitudinal component out, so there it
counts.

Co-Authored-By: Claude Opus 5 <noreply@anthropic.com>

File: src/albomb_description/urdf/albomb_sensors.xacro (robot description, xacro)
@@ -10,5 +10,8 @@
     </visual>
   </link>
-  <!-- VESC 6 MkVI onboard IMU. Yaw +90 deg; no roll.
+  <!-- VESC 6 MkVI onboard IMU. Yaw -90 deg; no roll.
+       The board is mounted turned 90 deg CLOCKWISE from the car's forward
+       direction, so the imu frame is -90 about z from base_link. Sign follows
+       from that directly: rpy rotates child vectors into the parent.
        The chip is mounted upside down on the board, but the FIRMWARE already
        corrects for that, so the data reaching us is Z up. Measured, level and
@@ -29,8 +32,17 @@
        Reading that + as "the board is upside down" is what put roll=pi in here
        once. Judge this from the topic, never from the tool.
-       STILL UNVERIFIED is +90 vs -90, which this static reading cannot show
-       and which only sets the longitudinal axis, not the yaw rate. At +90,
-       forward = -imu.y, so accelerating forwards should drive imu.y negative.
-       If it goes positive, this is -1.5708.
+       With no roll and yaw -90 the axes are
+           forward = +imu.y    left = -imu.x    up = +imu.z
+       Confirm by pushing the car forwards: imu.y should go POSITIVE. (This
+       spent a while at +1.5708, from believing Z faced the floor. It is worth
+       knowing that Rz(+90)Rx(180) and Rz(-90) give the same forward axis, so
+       that combination was self-consistent right up until the accelerometer
+       showed Z was up.)
+       The yaw does not reach cartographer: it tracks in this frame and
+       publishes base_link, so a constant rotation between imu and laser is
+       applied and then taken back off, and 2D uses only gyro z, which a yaw
+       rotation leaves alone. Maps made before this was corrected are fine.
+       controller_manager is different - it reads the longitudinal component
+       out, so there the yaw matters.
        VESC Tool's own Imu Rotation (roll 7.4 / pitch -4.7 / yaw 0) is mounting
        tilt only. Leave the 90 out of it; this joint is where it belongs.
@@ -42,5 +54,5 @@
     <parent link="${car_name}/base_link"/>
     <child link="${car_name}/imu"/>
-    <origin xyz="0.07 0.0 ${wheel_radius+0.04}" rpy="0 0 1.5708"/>
+    <origin xyz="0.07 0.0 ${wheel_radius+0.04}" rpy="0 0 -1.5708"/>
   </joint>
   <link name="${car_name}/laser">
